File: version1.kicad_pcb (KiCad board)
At the start: 2 copper layers, 324.5 x 130.4 mm, 278 parts, among them J1 AVR-ISP-6, J2 Conn_01x04, SW1 SW_Push, SW10 SW_Push, SW11 SW_Push, SW12 SW_Push, SW13 SW_Push, SW14 SW_Push, SW15 SW_Push, SW16 SW_Push, SW17 SW_Push, SW18 SW_Push, SW19 SW_Push, SW2 SW_Push, SW20 SW_Push, SW21 SW_Push, SW22 SW_Push, SW23 SW_Push, SW24 SW_Push, SW25 SW_Push, SW26 SW_Push, SW27 SW_Push, SW28 SW_Push, SW29 SW_Push, SW3 SW_Push, SW30 SW_Push, SW31 SW_Push, SW32 SW_Push, SW33 SW_Push, SW34 SW_Push, SW35 SW_Push, SW36 SW_Push, SW37 SW_Push, SW38 SW_Push, SW39 SW_Push, SW4 SW_Push, SW40 SW_Push, SW41 SW_Push, SW42 SW_Push, SW43 SW_Push, SW44 SW_Push, SW45 SW_Push, SW46 SW_Push, SW47 SW_Push, SW48 SW_Push, SW49 SW_Push, SW5 SW_Push, SW50 SW_Push, SW51 SW_Push, SW52 SW_Push, SW53 SW_Push, SW54 SW_Push, SW55 SW_Push, SW56 SW_Push, SW57 SW_Push, SW58 SW_Push, SW59 SW_Push, SW6 SW_Push, SW60 SW_Push, SW61 SW_Push, SW62 SW_Push, SW63 SW_Push, SW64 SW_Push, SW65 SW_Push, SW66 SW_Push, SW67 SW_Push, SW68 SW_Push, SW69 SW_Push, SW7 SW_Push, SW70 SW_Push, SW71 SW_Push, SW72 SW_Push, SW73 SW_Push, SW74 SW_Push, SW75 SW_Push, SW76 SW_Push, SW77 SW_Push, SW78 SW_Push, SW79 SW_Push, SW8 SW_Push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

Commit message: Final version
Parts:
- removed H6: MountingHole, MountingHole:MountingHole_3.5mm
- D1, D10, D11, D12, D13, D14, D15, D16, D17, D18, D19, D2, D20, D21, D22, D23, D24, D25, D26, D27, D28, D29, D3, D30, D31, D32, D33, D34, D35, D36, D37, D38, D39, D4, D40, D41, D42, D43, D44, D45, D46, D47, D48, D49, D5, D50, D51, D52, D53, D54, D55, D56, D57, D58, D59, D6, D60, D61, D62, D63, D64, D65, D66, D67, D68, D69, D7, D70, D71, D72, D73, D74, D75, D76, D77, D78, D79, D8, D80, D9: footprint Diode_SMD:D_0603_1608Metric_Pad1.05x0.95mm_HandSolder -> Diode_SMD:D_SOD-323_HandSoldering
- F1: footprint Fuse:Fuse_0603_1608Metric_Pad1.05x0.95mm_HandSolder -> Fuse:Fuse_1206_3216Metric_Pad1.42x1.75mm_HandSolder
- RE1: footprint Rotary_Encoder:RotaryEncoder_Alps_EC11E-Switch_Vertical_H20mm_CircularMountingHoles -> Rotary_Encoder:RotaryEncoder_Alps_EC11E-Switch_Vertical_H20mm
- SW1: footprint Button_Switch_SMD:SW_SPST_SKQG_WithStem -> Button_Switch_SMD:SW_Push_SPST_NO_Alps_SKRK
- SW10, SW11, SW12, SW13, SW14, SW15, SW16, SW17, SW18, SW19, SW2, SW20, SW21, SW22, SW23, SW24, SW25, SW26, SW27, SW3, SW30, SW31, SW32, SW33, SW34, SW35, SW36, SW37, SW38, SW39, SW4, SW40, SW41, SW44, SW45, SW46, SW47, SW48, SW49, SW5, SW50, SW51, SW52, SW53, SW54, SW56, SW58, SW59, SW6, SW60, SW61, SW62, SW63, SW64, SW65, SW66, SW67, SW69, SW7, SW70, SW75, SW76, SW77, SW78, SW79, SW8, SW80, SW9: footprint MX_Alps_Hybrid:MX-1U-NoLED -> MX_Only:MXOnly-1U-Hotswap
- SW28: footprint MX_Alps_Hybrid:MX-2U-NoLED -> MX_Only:MXOnly-2U-Hotswap
- SW29, SW42: footprint MX_Alps_Hybrid:MX-1.5U-NoLED -> MX_Only:MXOnly-1.5U-Hotswap
- SW43, SW68: footprint MX_Alps_Hybrid:MX-1.75U-NoLED -> MX_Only:MXOnly-1.75U-Hotswap
- SW55, SW57: footprint MX_Alps_Hybrid:MX-2.25U-NoLED -> MX_Only:MXOnly-2.25U-Hotswap
- SW71, SW72, SW73: footprint MX_Alps_Hybrid:MX-1.25U-NoLED -> MX_Only:MXOnly-1.25U-Hotswap
- SW74: footprint MX_Alps_Hybrid:MX-6.25U-NoLED -> MX_Only:MXOnly-6.25U-Hotswap-ReversedStabilizers
- moved H2 186.4 mm to (397.8, 83.8)
- moved H3 158.9 mm to (327.4, 154.9)
- moved H1 153.9 mm to (180.3, 193.0)
- moved H5 111.4 mm to (103.9, 83.8)
- moved H4 45.7 mm to (189.5, 83.8)
- moved C7 13.4 mm to (383.3, 121.8), turned to 90 degrees
- moved C10 12.6 mm to (371.3, 125.2), turned to 270 degrees
- moved C4 7.37 mm to (223.3, 191.3), turned to 180 degrees
- moved C3 6.04 mm to (223.3, 193.0), turned to 180 degrees
- moved C5 3.31 mm to (234.7, 184.9), turned to 270 degrees
- moved C6 1.55 mm to (236.5, 184.9), turned to 270 degrees
- moved D74 1.44 mm to (218.9, 195.6)
- moved D14 0.77 mm to (376.7, 83.8)
- moved R2 0.71 mm to (240.7, 197.9)
- moved R3 0.66 mm to (240.7, 195.6)
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Connections:
- SW10 pad 1: Net-(D9-Pad2) -> col8
- SW10 pad 2: col8 -> Net-(D9-Pad2)
- SW11 pad 1: Net-(D10-Pad2) -> col9
- SW11 pad 2: col9 -> Net-(D10-Pad2)
- SW12 pad 1: Net-(D11-Pad2) -> col10
- SW12 pad 2: col10 -> Net-(D11-Pad2)
- SW13 pad 1: Net-(D12-Pad2) -> col11
- SW13 pad 2: col11 -> Net-(D12-Pad2)
- SW14 pad 1: Net-(D13-Pad2) -> col12
- SW14 pad 2: col12 -> Net-(D13-Pad2)
- SW15 pad 1: Net-(D15-Pad2) -> col0
- SW15 pad 2: col0 -> Net-(D15-Pad2)
- SW16 pad 1: Net-(D16-Pad2) -> col1
- SW16 pad 2: col1 -> Net-(D16-Pad2)
- SW17 pad 1: Net-(D17-Pad2) -> col2
- SW17 pad 2: col2 -> Net-(D17-Pad2)
- SW18 pad 1: Net-(D18-Pad2) -> col3
- SW18 pad 2: col3 -> Net-(D18-Pad2)
- SW19 pad 1: Net-(D19-Pad2) -> col4
- SW19 pad 2: col4 -> Net-(D19-Pad2)
- SW2 pad 1: Net-(D1-Pad2) -> col0
- SW2 pad 2: col0 -> Net-(D1-Pad2)
- SW20 pad 1: Net-(D20-Pad2) -> col5
- SW20 pad 2: col5 -> Net-(D20-Pad2)
- SW21 pad 1: Net-(D21-Pad2) -> col6
- SW21 pad 2: col6 -> Net-(D21-Pad2)
- SW22 pad 1: Net-(D22-Pad2) -> col7
- SW22 pad 2: col7 -> Net-(D22-Pad2)
- SW23 pad 1: Net-(D23-Pad2) -> col8
- SW23 pad 2: col8 -> Net-(D23-Pad2)
- SW24 pad 1: Net-(D24-Pad2) -> col9
- SW24 pad 2: col9 -> Net-(D24-Pad2)
- SW25 pad 1: Net-(D25-Pad2) -> col10
- SW25 pad 2: col10 -> Net-(D25-Pad2)
- SW26 pad 1: Net-(D26-Pad2) -> col11
- SW26 pad 2: col11 -> Net-(D26-Pad2)
- SW27 pad 1: Net-(D27-Pad2) -> col12
- SW27 pad 2: col12 -> Net-(D27-Pad2)
- SW28 pad 1: Net-(D28-Pad2) -> col13
- SW28 pad 2: col13 -> Net-(D28-Pad2)
- SW29 pad 1: Net-(D29-Pad2) -> col0
- SW29 pad 2: col0 -> Net-(D29-Pad2)
- SW3 pad 1: Net-(D2-Pad2) -> col1
- SW3 pad 2: col1 -> Net-(D2-Pad2)
- SW30 pad 1: Net-(D30-Pad2) -> col1
- SW30 pad 2: col1 -> Net-(D30-Pad2)
- SW31 pad 1: Net-(D31-Pad2) -> col2
- SW31 pad 2: col2 -> Net-(D31-Pad2)
- SW32 pad 1: Net-(D32-Pad2) -> col3
- SW32 pad 2: col3 -> Net-(D32-Pad2)
- SW33 pad 1: Net-(D33-Pad2) -> col4
- SW33 pad 2: col4 -> Net-(D33-Pad2)
- SW34 pad 1: Net-(D34-Pad2) -> col5
- SW34 pad 2: col5 -> Net-(D34-Pad2)
- SW35 pad 1: Net-(D35-Pad2) -> col6
- SW35 pad 2: col6 -> Net-(D35-Pad2)
- SW36 pad 1: Net-(D36-Pad2) -> col7
- SW36 pad 2: col7 -> Net-(D36-Pad2)
- SW37 pad 1: Net-(D37-Pad2) -> col8
- SW37 pad 2: col8 -> Net-(D37-Pad2)
- SW38 pad 1: Net-(D38-Pad2) -> col9
- SW38 pad 2: col9 -> Net-(D38-Pad2)
- SW39 pad 1: Net-(D39-Pad2) -> col10
- SW39 pad 2: col10 -> Net-(D39-Pad2)
- SW4 pad 1: Net-(D3-Pad2) -> col2
- SW4 pad 2: col2 -> Net-(D3-Pad2)
- SW40 pad 1: Net-(D40-Pad2) -> col11
- SW40 pad 2: col11 -> Net-(D40-Pad2)
- SW41 pad 1: Net-(D41-Pad2) -> col12
- SW41 pad 2: col12 -> Net-(D41-Pad2)
- SW42 pad 1: Net-(D42-Pad2) -> col13
- SW42 pad 2: col13 -> Net-(D42-Pad2)
- SW43 pad 1: Net-(D43-Pad2) -> col0
- SW43 pad 2: col0 -> Net-(D43-Pad2)
- SW44 pad 1: Net-(D44-Pad2) -> col1
- SW44 pad 2: col1 -> Net-(D44-Pad2)
- SW45 pad 1: Net-(D45-Pad2) -> col2
- SW45 pad 2: col2 -> Net-(D45-Pad2)
- SW46 pad 1: Net-(D46-Pad2) -> col3
- SW46 pad 2: col3 -> Net-(D46-Pad2)
- SW47 pad 1: Net-(D47-Pad2) -> col4
- SW47 pad 2: col4 -> Net-(D47-Pad2)
- SW48 pad 1: Net-(D48-Pad2) -> col5
- SW48 pad 2: col5 -> Net-(D48-Pad2)
- SW49 pad 1: Net-(D49-Pad2) -> col6
- SW49 pad 2: col6 -> Net-(D49-Pad2)
- SW5 pad 1: Net-(D4-Pad2) -> col3
- SW5 pad 2: col3 -> Net-(D4-Pad2)
- SW50 pad 1: Net-(D50-Pad2) -> col7
- SW50 pad 2: col7 -> Net-(D50-Pad2)
- SW51 pad 1: Net-(D51-Pad2) -> col8
- SW51 pad 2: col8 -> Net-(D51-Pad2)
- SW52 pad 1: Net-(D52-Pad2) -> col9
- SW52 pad 2: col9 -> Net-(D52-Pad2)
- SW53 pad 1: Net-(D53-Pad2) -> col10
- SW53 pad 2: col10 -> Net-(D53-Pad2)
- SW54 pad 1: Net-(D54-Pad2) -> col11
- SW54 pad 2: col11 -> Net-(D54-Pad2)
- SW55 pad 1: Net-(D55-Pad2) -> col12
- SW55 pad 2: col12 -> Net-(D55-Pad2)
- SW56 pad 1: Net-(D56-Pad2) -> col13
- SW56 pad 2: col13 -> Net-(D56-Pad2)
- SW57 pad 1: Net-(D57-Pad2) -> col0
- SW57 pad 2: col0 -> Net-(D57-Pad2)
- SW58 pad 1: Net-(D58-Pad2) -> col1
- SW58 pad 2: col1 -> Net-(D58-Pad2)
- SW59 pad 1: Net-(D59-Pad2) -> col2
- SW59 pad 2: col2 -> Net-(D59-Pad2)
- SW6 pad 1: Net-(D5-Pad2) -> col4
- SW6 pad 2: col4 -> Net-(D5-Pad2)
- SW60 pad 1: Net-(D60-Pad2) -> col3
- SW60 pad 2: col3 -> Net-(D60-Pad2)
- SW61 pad 1: Net-(D61-Pad2) -> col4
- SW61 pad 2: col4 -> Net-(D61-Pad2)
- SW62 pad 1: Net-(D62-Pad2) -> col5
- SW62 pad 2: col5 -> Net-(D62-Pad2)
- SW63 pad 1: Net-(D63-Pad2) -> col6
- SW63 pad 2: col6 -> Net-(D63-Pad2)
- SW64 pad 1: Net-(D64-Pad2) -> col7
- SW64 pad 2: col7 -> Net-(D64-Pad2)
- SW65 pad 1: Net-(D65-Pad2) -> col8
- SW65 pad 2: col8 -> Net-(D65-Pad2)
- SW66 pad 1: Net-(D66-Pad2) -> col9
- SW66 pad 2: col9 -> Net-(D66-Pad2)
- SW67 pad 1: Net-(D67-Pad2) -> col10
- SW67 pad 2: col10 -> Net-(D67-Pad2)
- SW68 pad 1: Net-(D68-Pad2) -> col11
- SW68 pad 2: col11 -> Net-(D68-Pad2)
- SW69 pad 1: Net-(D69-Pad2) -> col12
- SW69 pad 2: col12 -> Net-(D69-Pad2)
- SW7 pad 1: Net-(D6-Pad2) -> col5
- SW7 pad 2: col5 -> Net-(D6-Pad2)
- SW70 pad 1: Net-(D70-Pad2) -> col13
- SW70 pad 2: col13 -> Net-(D70-Pad2)
- SW71 pad 1: Net-(D71-Pad2) -> col0
- SW71 pad 2: col0 -> Net-(D71-Pad2)
- SW72 pad 1: Net-(D72-Pad2) -> col1
- SW72 pad 2: col1 -> Net-(D72-Pad2)
- SW73 pad 1: Net-(D73-Pad2) -> col2
- SW73 pad 2: col2 -> Net-(D73-Pad2)
- SW74 pad 1: Net-(D74-Pad2) -> col5
- SW74 pad 2: col5 -> Net-(D74-Pad2)
- SW75 pad 1: Net-(D75-Pad2) -> col8
- SW75 pad 2: col8 -> Net-(D75-Pad2)
- SW76 pad 1: Net-(D76-Pad2) -> col9
- SW76 pad 2: col9 -> Net-(D76-Pad2)
- SW77 pad 1: Net-(D77-Pad2) -> col10
- SW77 pad 2: col10 -> Net-(D77-Pad2)
- SW78 pad 1: Net-(D78-Pad2) -> col11
- SW78 pad 2: col11 -> Net-(D78-Pad2)
- SW79 pad 1: Net-(D79-Pad2) -> col12
- SW79 pad 2: col12 -> Net-(D79-Pad2)
- SW8 pad 1: Net-(D7-Pad2) -> col6
- SW8 pad 2: col6 -> Net-(D7-Pad2)
- SW80 pad 1: Net-(D80-Pad2) -> col13
- SW80 pad 2: col13 -> Net-(D80-Pad2)
- SW9 pad 1: Net-(D8-Pad2) -> col7
- SW9 pad 2: col7 -> Net-(D8-Pad2)
Routing:
- net col9: track 256.4 -> 323.6 mm, vias 1 -> 6
- net col6: track 281.2 -> 347.9 mm, vias 1 -> 5
- net col5: track 320.2 -> 386.7 mm, vias 1 -> 6
- net col8: track 274.2 -> 340.5 mm, vias 1 -> 6
- net col13: track 183.5 -> 244.9 mm, vias 1 -> 10
- net col7: track 263.6 -> 323.8 mm, vias 1 -> 5
- net col10: track 244.3 -> 303.6 mm, vias 1 -> 6
- net col4: track 319.7 -> 378.0 mm, vias 1 -> 5
- net col2: track 385.9 -> 443.9 mm, vias 1 -> 6
- net col1: track 409.9 -> 466.8 mm, vias 1 -> 6
- net col3: track 338.7 -> 394.5 mm, vias 1 -> 5
- net col11: track 239.3 -> 291.8 mm, vias 1 -> 6
- net col0: track 423.7 -> 474.9 mm, vias 1 -> 6
- net col12: track 226.8 -> 273.6 mm, vias 1 -> 6
- net SW3: track 351.5 -> 390.5 mm
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Other:
- board size 324.5 x 130.4 mm -> 327.7 x 137.2 mm
- board text added: "JLCJLCJLCJLC"
- board text added: "Made by Dakota Paxton :)"
