File: version1.sch (KiCad schematic (older format))
At the start: 39 parts, among them J1 AVR-ISP-6, J2 Conn_01x04, SW1 SW_Push, U1 AT90USB1286-AU, U2 IS31FL3733-TQ, U3 PRTR5V0U2X, Y1 16Mhz

Commit message: Final version
Parts:
- removed H6: MountingHole, MountingHole:MountingHole_3.5mm, symbol Mechanical:MountingHole
- C2, C4, C6: value .1uF -> 0.1uF
Changed lines of the file:
@@
-$EndComp
-$Comp
-L Mechanical:MountingHole H6
-U 1 1 6075CF2B
-P 6950 7400
-F 0 "H6" H 7050 7446 50  0000 L CNN
-F 1 "MountingHole" H 7050 7355 50  0000 L CNN
-F 2 "MountingHole:MountingHole_3.5mm" H 6950 7400 50  0001 C CNN
-F 3 "~" H 6950 7400 50  0001 C CNN
-	1    6950 7400
-	1    0    0    -1
 $EndComp
 $Comp
@@
 Text GLabel 11250 2600 2    50   Input ~ 0
 CS2
-Text GLabel 11250 2500 2    50   Input ~ 0
-CS1
 Connection ~ 10450 5600
 Wire Wire Line
@@
 P 11000 1850
 F 0 "C4" H 11092 1896 50  0000 L CNN
-F 1 ".1uF" H 11092 1805 50  0000 L CNN
+F 1 "0.1uF" H 11092 1805 50  0000 L CNN
 F 2 "Capacitor_SMD:C_0603_1608Metric_Pad1.08x0.95mm_HandSolder" H 11000 1850 50  0001 C CNN
 F 3 "~" H 11000 1850 50  0001 C CNN
@@
 P 10150 1850
 F 0 "C2" H 10242 1896 50  0000 L CNN
-F 1 ".1uF" H 10242 1805 50  0000 L CNN
+F 1 "0.1uF" H 10242 1805 50  0000 L CNN
 F 2 "Capacitor_SMD:C_0603_1608Metric_Pad1.08x0.95mm_HandSolder" H 10150 1850 50  0001 C CNN
 F 3 "~" H 10150 1850 50  0001 C CNN
@@
 P 11700 1850
 F 0 "C6" H 11792 1896 50  0000 L CNN
-F 1 ".1uF" H 11792 1805 50  0000 L CNN
+F 1 "0.1uF" H 11792 1805 50  0000 L CNN
 F 2 "Capacitor_SMD:C_0603_1608Metric_Pad1.08x0.95mm_HandSolder" H 11700 1850 50  0001 C CNN
 F 3 "~" H 11700 1850 50  0001 C CNN
@@
 NoConn ~ 11250 4800
 NoConn ~ 11250 4900
-NoConn ~ 11250 5000
-NoConn ~ 11250 5100
-NoConn ~ 11250 5200
-NoConn ~ 11250 5300
 NoConn ~ 9850 2900
 NoConn ~ 9850 3300
@@
 Text GLabel 2500 5650 1    50   Input ~ 0
 DN
+NoConn ~ 11250 5000
+NoConn ~ 11250 5300
+NoConn ~ 11250 5200
+NoConn ~ 11250 5100
+Text GLabel 11250 2500 2    50   Input ~ 0
+CS1
 $EndSCHEMATC
